Commit message: cube_petit.xacroの編集

File: cube_petit/urdf/cube_petit.old.xacro (robot description, xacro)
@@ -5,5 +5,5 @@
     <parent link="base_link"/>
     <child link="body_link"/>
-    <origin rpy="0 0 0" xyz="0 0 0"/>
+    <origin rpy="0 0 0" xyz="0.0 0 0"/>
   </joint>
   <link name="body_link">
@@ -41,5 +41,5 @@
     <parent link="body_link"/>
     <child link="pacecat_link"/>
-    <origin rpy="0 0 3.14159" xyz="0.0 0 0.23975"/>
+    <origin rpy="0 0 0" xyz="0.0 0 0.23975"/>
   </joint>
   <link name="pacecat_link">
@@ -154,4 +154,5 @@
     <!-- <limit effort="1000" velocity=""/> -->
   </joint>
+  <!-- only for gazebo -->
   <transmission name="right_wheel_trans" type="SimpleTransmission">
     <type>transmission_interface/SimpleTransmission</type>
@@ -194,4 +195,5 @@
     <kd value="0"/>
   </gazebo>
+  <!-- load gazebo plugin (hardware interface) -->
   <gazebo>
     <plugin name="gazebo_ros_control" filename="libgazebo_ros_control.so">
