Commit message: cube_petit_descriptionパッケージの作成
cube-petit本体のxacroファイル

File: cube_petit_description/urdf/cube_petit.xacro (robot description, xacro)
@@ -11,5 +11,5 @@
       <origin rpy="0 0 0" xyz="0 0 0"/>
       <geometry>
-    	  <mesh filename="package://cube_petit/meshes/cube_petit/cube_petit_body.obj"/>
+    	  <mesh filename="package://cube_petit_description/meshes/cube_petit/cube_petit_body.obj"/>
       </geometry>
     </visual>
@@ -225,5 +225,5 @@
     <origin rpy="-1.57079632679 0 0" xyz="0 0 0"/>
       <geometry>
-	      <mesh filename="package://cube_petit/meshes/cube_petit/cube_petit_wheel.obj"/>
+	      <mesh filename="package://cube_petit_description/meshes/cube_petit/cube_petit_wheel.obj"/>
       </geometry>
     </visual>
@@ -272,5 +272,5 @@
       <origin rpy="1.57079632679 0 0" xyz="0 0 0"/>
       <geometry>
-        <mesh filename="package://cube_petit/meshes/cube_petit/cube_petit_wheel.obj"/>
+        <mesh filename="package://cube_petit_description/meshes/cube_petit/cube_petit_wheel.obj"/>
       </geometry>
     </visual>

Commit message: cube_petit.xacroの修正 複数xacroファイルに分ける

File: cube_petit_description/urdf/cube_petit.xacro (robot description, xacro)
@@ -38,257 +38,7 @@
     <kd value="0"/>
   </gazebo>
-  <joint name="laser_joint" type="fixed">
-    <parent link="body_link"/>
-    <child link="pacecat_link"/>
-    <origin rpy="0 0 3.14159" xyz="0.0 0 0.23975"/>
-  </joint>
-  <link name="pacecat_link">
-    <inertial>
-      <origin rpy="0 0 0" xyz="0.00000000 0.00000000 0.00208424"/>
-      <mass value="0.11166745"/>
-      <inertia
-        ixx="0.004391"
-        ixy="0.000000" iyy="0.004391"
-        ixz="0.000000" iyz="0.000000" izz="0.004277"/>
-    </inertial>
-    <visual>
-      <origin rpy="0 0 0" xyz="0 0 0"/>
-      <geometry>
-        <cylinder length="0.0315" radius="0.025"/>
-      </geometry>
-      <material name="red"/>
-    </visual>
-    <collision>
-      <origin rpy="0 0 0" xyz="0 0 0"/>
-      <geometry>
-        <cylinder length="0.0315" radius="0.025"/>
-      </geometry>
-    </collision>
-  </link>
-  <gazebo reference="pacecat_link">
-    <mu1 value="0.5"/>
-    <kp value="50000"/>
-    <kd value="0"/>
-    <sensor type="ray" name="pacecat">
-      <pose>0 0 0 0 0 0</pose>
-      <visualize>false</visualize>
-      <update_rate>10</update_rate>
-      <ray>
-        <scan>
-          <horizontal>
-            <samples>400</samples>
-            <resolution>1</resolution>
-            <min_angle>${radians(-180)}</min_angle>
-            <max_angle>${radians( 180)}</max_angle>
-          </horizontal>
-        </scan>
-        <range>
-          <min>0.16</min>
-          <max>20.0</max>
-          <resolution>0.01</resolution>
-        </range>
-        <noise>
-          <type>gaussian</type>
-          <mean>0.0</mean>
-          <stddev>0.01</stddev>
-        </noise>
-      </ray>
-      <plugin name="gazebo_ros_lidar_controller" filename="libgazebo_ros_laser.so">
-        <topicName>/pacecat/scan</topicName>
-        <frameName>pacecat_link</frameName>
-      </plugin>
-    </sensor>
-  </gazebo>
-  <joint name="depth_joint" type="fixed">
-    <parent link="body_link"/>
-    <child link="camera_link"/>
-    <origin rpy="0 0.0034 0" xyz="0.10137 0.0 0.10306"/>
-  </joint>
-  <link name="camera_link">
-    <inertial>
-      <origin rpy="0 0 0" xyz="0.00000000 0.00000000 0.0000000"/>
-      <mass value="0.11166745"/>
-      <inertia
-        ixx="0.004391"
-        ixy="0.000000" iyy="0.004391"
-        ixz="0.000000" iyz="0.000000" izz="0.004277"/>
-    </inertial>
-    <visual>
-      <origin rpy="0 0 0" xyz="0 0 0"/>
-      <geometry>
-        <cylinder length="0.001" radius="0.001"/>
-      </geometry>
-      <material name="red"/>
-    </visual>
-    <collision>
-      <origin rpy="0 0 0" xyz="0 0 0"/>
-      <geometry>
-        <cylinder length="0.001" radius="0.001"/>
-      </geometry>
-    </collision>
-  </link>
-  <gazebo reference="camera_link">
-    <mu1 value="0.5"/>
-    <kp value="50000"/>
-    <kd value="0"/>
-    <sensor type="depth" name="camera">
-      <always_on>true</always_on>
-      <update_rate>4.0</update_rate>
-      <camera>
-        <horizontal_fov>${60.0*3.1415926/180.0}</horizontal_fov>
-        <image>
-          <format>R8G8B8</format>
-          <width>640</width>
-          <height>480</height>
-        </image>
-        <clip>
-          <near>0.2</near>
-          <far>1.5</far>
-        </clip>
-      </camera>
-      <plugin name="kinect_camera_controller" filename="libgazebo_ros_openni_kinect.so">
-      <!-- <plugin name="realsense_camera_controller" filename="libRealSensePlugin.so"> -->
-        <cameraName>camera</cameraName>
-        <alwaysOn>true</alwaysOn>
-        <updateRate>4</updateRate>
-        <imageTopicName>camera/image_color</imageTopicName>
-        <depthImageTopicName>camera/image_depth_rect</depthImageTopicName>
-        <pointCloudTopicName>camera/points</pointCloudTopicName>
-        <cameraInfoTopicName>camera/camera_info</cameraInfoTopicName>
-        <!-- <depthImageCameraInfoTopicName>depth/camera_info</depthImageCameraInfoTopicName> -->
-        <frameName>camera_optical_link</frameName>
-        <pointCloudCutoff>0.2</pointCloudCutoff>
-        <pointCloudCutoffMax>1.5</pointCloudCutoffMax>
-        <baseline>0.1</baseline>
-        <distortion_k1>0.0</distortion_k1>
-        <distortion_k2>0.0</distortion_k2>
-        <distortion_k3>0.0</distortion_k3>
-        <distortion_t1>0.0</distortion_t1>
-        <distortion_t2>0.0</distortion_t2>
-      </plugin>
-    </sensor>
-  </gazebo>
-  <joint name="depth_optical_joint" type="fixed">
-    <parent link="camera_link"/>
-    <child link="camera_optical_link"/>
-    <origin rpy="-1.57 0 -1.57" xyz="0.0 0.0 0.0"/>
-  </joint>
-  <link name="camera_optical_link">
-    <inertial>
-      <origin rpy="0 0 0" xyz="0.00000000 0.00000000 0.0000000"/>
-      <mass value="0.11166745"/>
-      <inertia
-        ixx="0.004391"
-        ixy="0.000000" iyy="0.004391"
-        ixz="0.000000" iyz="0.000000" izz="0.004277"/>
-    </inertial>
-    <visual>
-      <origin rpy="0 0 0" xyz="0 0 0"/>
-      <geometry>
-        <cylinder length="0.001" radius="0.001"/>
-      </geometry>
-      <material name="red"/>
-    </visual>
-    <collision>
-      <origin rpy="0 0 0" xyz="0 0 0"/>
-      <geometry>
-        <cylinder length="0.001" radius="0.001"/>
-      </geometry>
-    </collision>
-  </link>
-  <joint name="left_wheel_joint" type="continuous">
-    <origin rpy="0 0 0" xyz="-0.002 0.077 0.033"/>
-    <parent link="body_link"/>
-    <child link="left_wheel_link"/>
-    <axis xyz="0 1 0"/>
-    <!-- <limit effort="1000"/> -->
-  </joint>
-  <transmission name="left_wheel_trans" type="SimpleTransmission">
-    <type>transmission_interface/SimpleTransmission</type>
-    <actuator name="left_wheel_motor">
-      <mechanicalReduction>1</mechanicalReduction>
-    </actuator>
-    <joint name="left_wheel_joint">
-      <hardwareInterface>hardware_interface/VelocityJointInterface</hardwareInterface>
-    </joint>
-  </transmission>
-  <link name="left_wheel_link">
-    <inertial>
-      <origin rpy="0 0 0" xyz="-0.00000147 0.00093592 -0.00000239"/>
-      <mass value="0.2986774"/>
-      <inertia
-        ixx="0.0001147"
-        ixy="0.00000000" iyy="0.0002130"
-        ixz="0.00000000" iyz="0.0000001" izz="0.0001148"/>
-    </inertial>
-    <visual>
-    <origin rpy="-1.57079632679 0 0" xyz="0 0 0"/>
-      <geometry>
-	      <mesh filename="package://cube_petit_description/meshes/cube_petit/cube_petit_wheel.obj"/>
-      </geometry>
-    </visual>
-    <collision>
-      <origin rpy="1.57079632679 0 0" xyz="0 0 0"/>
-      <geometry>
-        <cylinder length="0.002" radius="0.033"/>
-      </geometry>
-    </collision>
-  </link>
-  <gazebo reference="left_wheel_link">
-    <selfCollide>false</selfCollide>
-    <maxContacts>2</maxContacts>
-    <minDepth>0</minDepth>
-    <!-- <dampingFactor>0</dampingFactor> -->
-    <mu1 value="2.5"/>
-    <kp value="50000"/>
-    <kd value="0"/>
-  </gazebo>
-  <joint name="right_wheel_joint" type="continuous">
-    <origin rpy="0 0 0" xyz="-0.002 -0.077 0.033"/>
-    <parent link="body_link"/>
-    <child link="right_wheel_link"/>
-    <axis xyz="0 1 0"/>
-    <!-- <limit effort="1000" velocity=""/> -->
-  </joint>
-  <transmission name="right_wheel_trans" type="SimpleTransmission">
-    <type>transmission_interface/SimpleTransmission</type>
-    <actuator name="right_wheel_motor">
-      <mechanicalReduction>1</mechanicalReduction>
-    </actuator>
-    <joint name="right_wheel_joint">
-      <hardwareInterface>hardware_interface/VelocityJointInterface</hardwareInterface>
-    </joint>
-  </transmission>
-  <link name="right_wheel_link">
-    <inertial>
-      <origin rpy="0 0 0" xyz="-0.00000147 0.00093592 -0.00000239"/>
-      <mass value="0.2986774"/>
-      <inertia
-        ixx="0.0001147"
-        ixy="0.00000000" iyy="0.0002130"
-        ixz="0.00000000" iyz="0.0000001" izz="0.0001148"/>
-    </inertial>
-    <visual>
-      <origin rpy="1.57079632679 0 0" xyz="0 0 0"/>
-      <geometry>
-        <mesh filename="package://cube_petit_description/meshes/cube_petit/cube_petit_wheel.obj"/>
-      </geometry>
-    </visual>
-    <collision>
-      <origin rpy="1.57079632679 0 0" xyz="0 0 0"/>
-      <geometry>
-        <cylinder length="0.002" radius="0.033"/>
-      </geometry>
-    </collision>
-  </link>
-  <gazebo reference="right_wheel_link">
-    <selfCollide>false</selfCollide>
-    <maxContacts>2</maxContacts>
-    <minDepth>0</minDepth>
-    <!-- <dampingFactor>0</dampingFactor> -->
-    <mu1 value="2.5"/>
-    <kp value="50000"/>
-    <kd value="0"/>
-  </gazebo>
+  <xacro:include filename="$(find cube_petit_description)/urdf/sensors/lidar.xacro" />
+  <xacro:include filename="$(find cube_petit_description)/urdf/sensors/depth.xacro" />
+  <xacro:include filename="$(find cube_petit_description)/urdf/wheels/turtlebot_wheels.xacro" />
   <gazebo>
     <plugin name="gazebo_ros_control" filename="libgazebo_ros_control.so">
