Commit message: cube-petitのxacroにbrass batteryのＰｌｕｇｉｎを追加

File: cube_petit_description/urdf/cube_petit_v2.xacro (robot description, xacro)
@@ -1,4 +1,6 @@
 <?xml version="1.0" ?>
-<robot name="cube_petit" xmlns:xacro="http://ros.org/wiki/xacro">
+<robot name="cube_petit" xmlns:xacro="http://www.ros.org/wiki/xacro">
+  <xacro:include filename="$(find cube_petit_description)/xacro/publish_pose.xacro"/>
+  <xacro:include filename="$(find cube_petit_description)/xacro/brass_gazebo_battery.xacro"/>
   <link name="base_link"/>
   <joint name="body_joint" type="fixed">
@@ -38,4 +40,10 @@
     <kd value="0"/>
   </gazebo>
+  <link name="connector_link"/>
+  <joint name="connector_joint" type="fixed">
+    <parent link="base_link"/>
+    <child link="connector_link"/>
+    <origin rpy="0 0 3.14" xyz="-0.11 0 0.025"/>
+  </joint>
   <xacro:include filename="$(find cube_petit_description)/urdf/sensors/lidar.xacro" />
   <!-- rear camera -->
@@ -44,4 +52,7 @@
   <xacro:include filename="$(find cube_petit_description)/urdf/wheels/tamiya_wheels.xacro" />
   <!-- <xacro:include filename="$(find cube_petit_description)/urdf/wheels/turtlebot_wheels.xacro" /> -->
+  <!-- <xacro:brass_gazebo_battery_plugin parent_link="base_link" voltage="25.12" capacity_ah="2.0" charge_current="100.0" discharge_current="20.0" /> -->
+  <xacro:brass_gazebo_battery_plugin parent_link="base_link" voltage="15.12" capacity_ah="2.0" charge_current="100.0" discharge_current="20.0" />
+  <xacro:publish_pose_plugin link_name="base_link" topic_out="/gazebo/docking_station_simulation/robot_pose" update_rate="30" />
   <gazebo>
     <plugin name="gazebo_ros_control" filename="libgazebo_ros_control.so">

Commit message: ar_docking_controllerの修正、動く

File: cube_petit_description/urdf/cube_petit_v2.xacro (robot description, xacro)
@@ -8,4 +8,10 @@
     <child link="body_link"/>
     <origin rpy="0 0 0" xyz="0 0 0"/>
+  </joint>
+  <link name="base_link_reverse"/>
+  <joint name="base_link_reverse_joint" type="fixed">
+    <parent link="base_link"/>
+    <child link="base_link_reverse"/>
+    <origin rpy="0 0 3.1415926" xyz="0 0 0"/>
   </joint>
   <link name="body_link">

Commit message: add robot_pose

File: cube_petit_description/urdf/cube_petit_v2.xacro (robot description, xacro)
@@ -1,3 +1,3 @@
-<?xml version="1.0" ?>
+<?xml version="1.0"?>
 <robot name="cube_petit" xmlns:xacro="http://www.ros.org/wiki/xacro">
   <xacro:include filename="$(find cube_petit_description)/xacro/publish_pose.xacro"/>
@@ -19,5 +19,6 @@
       <origin rpy="0 0 0" xyz="0 0 0"/>
       <geometry>
-    	  <mesh filename="package://cube_petit_description/meshes/cube_petit/body/2/cube_petit_v2_body.obj"/>
+        <mesh
+          filename="package://cube_petit_description/meshes/cube_petit/body/2/cube_petit_v2_body.obj"/>
       </geometry>
     </visual>
@@ -52,13 +53,17 @@
     <origin rpy="0 0 3.14" xyz="-0.11 0 0.025"/>
   </joint>
-  <xacro:include filename="$(find cube_petit_description)/urdf/sensors/lidar.xacro" />
+  <xacro:include filename="$(find cube_petit_description)/urdf/sensors/lidar.xacro"/>
   <!-- rear camera -->
-  <xacro:include filename="$(find cube_petit_description)/urdf/sensors/camera.xacro" />
-  <xacro:include filename="$(find cube_petit_description)/urdf/sensors/depth.xacro" />
-  <xacro:include filename="$(find cube_petit_description)/urdf/wheels/tamiya_wheels.xacro" />
-  <!-- <xacro:include filename="$(find cube_petit_description)/urdf/wheels/turtlebot_wheels.xacro" /> -->
-  <!-- <xacro:brass_gazebo_battery_plugin parent_link="base_link" voltage="25.12" capacity_ah="2.0" charge_current="100.0" discharge_current="20.0" /> -->
-  <xacro:brass_gazebo_battery_plugin parent_link="base_link" voltage="15.12" capacity_ah="2.0" charge_current="100.0" discharge_current="20.0" />
-  <xacro:publish_pose_plugin link_name="base_link" topic_out="/gazebo/docking_station_simulation/robot_pose" update_rate="30" />
+  <xacro:include filename="$(find cube_petit_description)/urdf/sensors/camera.xacro"/>
+  <xacro:include filename="$(find cube_petit_description)/urdf/sensors/depth.xacro"/>
+  <xacro:include filename="$(find cube_petit_description)/urdf/wheels/tamiya_wheels.xacro"/>
+  <!-- <xacro:include filename="$(find cube_petit_description)/urdf/wheels/turtlebot_wheels.xacro"
+  /> -->
+  <!-- <xacro:brass_gazebo_battery_plugin parent_link="base_link" voltage="25.12" capacity_ah="2.0"
+  charge_current="100.0" discharge_current="20.0" /> -->
+  <xacro:brass_gazebo_battery_plugin parent_link="base_link" voltage="15.12" capacity_ah="2.0"
+    charge_current="100.0" discharge_current="20.0"/>
+  <xacro:publish_pose_plugin link_name="base_link"
+    topic_out="/gazebo/docking_station_simulation/robot_pose" update_rate="30"/>
   <gazebo>
     <plugin name="gazebo_ros_control" filename="libgazebo_ros_control.so">
@@ -67,3 +72,11 @@
     </plugin>
   </gazebo>
+  <gazebo>
+    <plugin name="base_link_pose_publisher_plugin" filename="libgazebo_ros_p3d.so">
+      <frameName>world</frameName>
+      <bodyName>base_link</bodyName>
+      <topicName>gazebo/robot_pose</topicName>
+      <updateRate>10</updateRate>
+    </plugin>
+  </gazebo>
 </robot>

Commit message: add omron, fix talk

File: cube_petit_description/urdf/cube_petit_v2.xacro (robot description, xacro)
@@ -14,4 +14,10 @@
     <child link="base_link_reverse"/>
     <origin rpy="0 0 3.1415926" xyz="0 0 0"/>
+  </joint>
+  <link name="respeaker_base"/>
+  <joint name="respeaker_joint" type="fixed">
+    <parent link="base_link"/>
+    <child link="respeaker_base"/>
+    <origin rpy="0 0 0" xyz="0 0 0.28"/>
   </joint>
   <link name="body_link">
@@ -53,7 +59,8 @@
     <origin rpy="0 0 3.14" xyz="-0.11 0 0.025"/>
   </joint>
-  <xacro:include filename="$(find cube_petit_description)/urdf/sensors/lidar.xacro"/>
+  <xacro:include filename="$(find cube_petit_description)/urdf/sensors/lidar.xacro" />
   <!-- rear camera -->
-  <xacro:include filename="$(find cube_petit_description)/urdf/sensors/camera.xacro"/>
+  <xacro:include filename="$(find cube_petit_description)/urdf/sensors/camera.xacro" />
+  <xacro:include filename="$(find cube_petit_description)/urdf/sensors/depth.xacro" />
   <xacro:include filename="$(find cube_petit_description)/urdf/sensors/depth.xacro"/>
   <xacro:include filename="$(find cube_petit_description)/urdf/wheels/tamiya_wheels.xacro"/>
