Commit message: base_linkからstation_base_linkに変更

File: cube_petit_gazebo/models/charge_doc/cube_petit_charge_doc.xacro (robot description, xacro)
@@ -4,7 +4,7 @@
 As a workaround, you can add an extra dummy link to your URDF. -->
 <robot name="charge_doc" xmlns:xacro="http://ros.org/wiki/xacro">
-  <link name="base_link"/>
+  <link name="station_base_link"/>
   <joint name="base_joint" type="fixed">
-    <parent link="base_link"/>
+    <parent link="station_base_link"/>
     <child link="charge_doc_base_link"/>
   </joint>
@@ -57,5 +57,5 @@
   <link name="charge_doc_base2_link"/> -->
   <!-- Gazebo Physical Parameters -->
-  <gazebo reference="charge_doc_base_link">
+  <gazebo reference="station_base_link">
     <!-- <kp>100000.0</kp>
     <kd>100.0</kd>
@@ -73,5 +73,5 @@
     <plugin name="publish_station_pose" filename="libgazebo_ros_p3d.so">
       <frameName>world</frameName>
-      <bodyName>charge_doc_base_link</bodyName>
+      <bodyName>station_base_link</bodyName>
       <topicName>/gazebo/docking_station_simulation/station_pose</topicName>
       <updateRate>30.0</updateRate>
