Commit message: lidar and slam

File: cube_petit_description/xacro/cube_petit_gazebo.xacro (robot description, xacro)
@@ -3,6 +3,8 @@
   <!-- General -->
   <!-- <xacro:include filename="color_property.xacro"/> -->
-  <!-- <xacro:include filename="$(find cube_petit_description)/xacro/publish_pose/publish_pose.xacro"/>
-  <xacro:include filename="$(find cube_petit_description)/xacro/brass_gazebo_battery/brass_gazebo_battery.xacro"/> -->
+  <!-- <xacro:include filename="$(find
+  cube_petit_description)/xacro/publish_pose/publish_pose.xacro"/>
+  <xacro:include filename="$(find
+  cube_petit_description)/xacro/brass_gazebo_battery/brass_gazebo_battery.xacro"/> -->
   <link name="base_link"/>
   <joint name="body_joint" type="fixed">
@@ -27,5 +29,6 @@
       <origin rpy="0 0 0" xyz="0 0 0"/>
       <geometry>
-        <mesh filename="file://$(find cube_petit_description)/meshes/cube_petit/body/2/cube_petit_v2_body.obj"/>
+        <mesh
+          filename="file://$(find cube_petit_description)/meshes/cube_petit/body/2/cube_petit_v2_body.obj"/>
       </geometry>
     </visual>
@@ -41,5 +44,6 @@
       <origin rpy="0 0 0" xyz="0.00440023 0.00053314 0.15283194"/>
       <mass value="1.98239086"/>
-      <inertia ixx="0.02351680" ixy="0.00001868" iyy="0.02505713" ixz="-0.00012952" iyz="-0.00004728" izz="0.02060399"/>
+      <inertia ixx="0.02351680" ixy="0.00001868" iyy="0.02505713" ixz="-0.00012952"
+        iyz="-0.00004728" izz="0.02060399"/>
     </inertial>
   </link>
@@ -57,5 +61,74 @@
     <origin rpy="0 0 3.14" xyz="-0.11 0 0.025"/>
   </joint>
-  <xacro:include filename="$(find cube_petit_description)/xacro/sensors/lidar.xacro"/>
+  <!-- lidar -->
+  <joint name="laser_joint" type="fixed">
+    <parent link="body_link"/>
+    <child link="pacecat_link"/>
+    <origin rpy="0 0 0" xyz="0.0 0 0.23975"/>
+  </joint>
+  <link name="pacecat_link">
+    <inertial>
+      <origin rpy="0 0 0" xyz="0.00000000 0.00000000 0.00208424"/>
+      <mass value="0.11166745"/>
+      <inertia
+        ixx="0.004391"
+        ixy="0.000000" iyy="0.004391"
+        ixz="0.000000" iyz="0.000000" izz="0.004277"/>
+    </inertial>
+    <visual>
+      <origin rpy="0 0 0" xyz="0 0 0"/>
+      <geometry>
+        <cylinder length="0.0315" radius="0.025"/>
+      </geometry>
+      <!-- <material name="red"/> -->
+    </visual>
+    <collision>
+      <origin rpy="0 0 0" xyz="0 0 0"/>
+      <geometry>
+        <cylinder length="0.0315" radius="0.025"/>
+      </geometry>
+    </collision>
+  </link>
+  <gazebo reference="pacecat_link">
+    <material>red</material>
+    <mu1>0.2</mu1>
+    <mu2>0.2</mu2>
+    <self_collide>false</self_collide>
+    <sensor type="ray" name="pacecat_ray">
+      <pose>0 0 0 0 0 0</pose>
+      <always_on>true</always_on>
+      <visualize>false</visualize>
+      <update_rate>10</update_rate>
+      <ray>
+        <scan>
+          <horizontal>
+            <samples>400</samples>
+            <resolution>1</resolution>
+            <min_angle>${radians(-180)}</min_angle>
+            <max_angle>${radians( 180)}</max_angle>
+          </horizontal>
+        </scan>
+        <range>
+          <min>0.16</min>
+          <max>20.0</max>
+          <resolution>0.01</resolution>
+        </range>
+        <noise>
+          <type>gaussian</type>
+          <mean>0.0</mean>
+          <stddev>0.01</stddev>
+        </noise>
+      </ray>
+      <plugin name="scan" filename="libgazebo_ros_ray_sensor.so">
+        <ros>
+          <!-- <namespace>/cube_petit</namespace> -->
+          <remapping>~/out:=scan</remapping>
+        </ros>
+        <output_type>sensor_msgs/LaserScan</output_type>
+        <frame_name>pacecat_link</frame_name>
+      </plugin>
+    </sensor>
+  </gazebo>
+  <!-- <xacro:include filename="$(find cube_petit_description)/xacro/sensors/lidar.xacro"/> -->
   <!-- rear camera -->
   <!-- <xacro:include filename="$(find cube_petit_description)/xacro/sensors/camera.xacro" /> -->
@@ -103,5 +176,6 @@
       <origin rpy="0 0 0" xyz="-0.00000147 0.00093592 -0.00000239"/>
       <mass value="0.2986774"/>
-      <inertia ixx="0.0001147" ixy="0.00000000" iyy="0.0002130" ixz="0.00000000" iyz="0.0000001" izz="0.0001148"/>
+      <inertia ixx="0.0001147" ixy="0.00000000" iyy="0.0002130" ixz="0.00000000" iyz="0.0000001"
+        izz="0.0001148"/>
     </inertial>
     <visual>
@@ -148,5 +222,6 @@
       <origin rpy="0 0 0" xyz="-0.00000147 0.00093592 -0.00000239"/>
       <mass value="0.2986774"/>
-      <inertia ixx="0.0001147" ixy="0.00000000" iyy="0.0002130" ixz="0.00000000" iyz="0.0000001" izz="0.0001148"/>
+      <inertia ixx="0.0001147" ixy="0.00000000" iyy="0.0002130" ixz="0.00000000" iyz="0.0000001"
+        izz="0.0001148"/>
     </inertial>
     <visual>

File: cube_petit_description/xacro/sensors/lidar.xacro (robot description, xacro)
@@ -34,6 +34,7 @@
     <kd value="0"/>
     <sensor type="gpu_ray" name="pacecat">
+      <alwaysOn>true</alwaysOn>
       <pose>0 0 0 0 0 0</pose>
-      <visualize>false</visualize>
+      <visualize>true</visualize>
       <update_rate>10</update_rate>
       <ray>
@@ -57,7 +58,11 @@
         </noise>
       </ray>
-      <plugin name="gazebo_ros_lidar_controller" filename="libgazebo_ros_gpu_laser.so">
-        <topicName>/pacecat/scan</topicName>
-        <frameName>pacecat_link</frameName>
+      <plugin name="gazebo_ros_laser" filename="libgazebo_ros_ray_sensor.so">
+        <ros>
+          <namespace>/pacecat</namespace>
+          <remapping>~/out:=/pacecat/scan</remapping>
+        </ros>
+        <output_type>sensor_msgs/LaserScan</output_type>
+        <frame_name>pacecat_link</frame_name>
       </plugin>
     </sensor>

Commit message: lidar and slam

File: cube_petit_description/xacro/cube_petit_gazebo.xacro (robot description, xacro)
@@ -29,6 +29,5 @@
       <origin rpy="0 0 0" xyz="0 0 0"/>
       <geometry>
-        <mesh
-          filename="file://$(find cube_petit_description)/meshes/cube_petit/body/2/cube_petit_v2_body.obj"/>
+        <mesh filename="file://$(find cube_petit_description)/meshes/cube_petit/body/2/cube_petit_v2_body.obj"/>
       </geometry>
     </visual>
@@ -44,6 +43,5 @@
       <origin rpy="0 0 0" xyz="0.00440023 0.00053314 0.15283194"/>
       <mass value="1.98239086"/>
-      <inertia ixx="0.02351680" ixy="0.00001868" iyy="0.02505713" ixz="-0.00012952"
-        iyz="-0.00004728" izz="0.02060399"/>
+      <inertia ixx="0.02351680" ixy="0.00001868" iyy="0.02505713" ixz="-0.00012952" iyz="-0.00004728" izz="0.02060399"/>
     </inertial>
   </link>
@@ -71,8 +69,5 @@
       <origin rpy="0 0 0" xyz="0.00000000 0.00000000 0.00208424"/>
       <mass value="0.11166745"/>
-      <inertia
-        ixx="0.004391"
-        ixy="0.000000" iyy="0.004391"
-        ixz="0.000000" iyz="0.000000" izz="0.004277"/>
+      <inertia ixx="0.004391" ixy="0.000000" iyy="0.004391" ixz="0.000000" iyz="0.000000" izz="0.004277"/>
     </inertial>
     <visual>
@@ -176,6 +171,5 @@
       <origin rpy="0 0 0" xyz="-0.00000147 0.00093592 -0.00000239"/>
       <mass value="0.2986774"/>
-      <inertia ixx="0.0001147" ixy="0.00000000" iyy="0.0002130" ixz="0.00000000" iyz="0.0000001"
-        izz="0.0001148"/>
+      <inertia ixx="0.0001147" ixy="0.00000000" iyy="0.0002130" ixz="0.00000000" iyz="0.0000001" izz="0.0001148"/>
     </inertial>
     <visual>
@@ -222,6 +216,5 @@
       <origin rpy="0 0 0" xyz="-0.00000147 0.00093592 -0.00000239"/>
       <mass value="0.2986774"/>
-      <inertia ixx="0.0001147" ixy="0.00000000" iyy="0.0002130" ixz="0.00000000" iyz="0.0000001"
-        izz="0.0001148"/>
+      <inertia ixx="0.0001147" ixy="0.00000000" iyy="0.0002130" ixz="0.00000000" iyz="0.0000001" izz="0.0001148"/>
     </inertial>
     <visual>

File: cube_petit_description/xacro/sensors/lidar.xacro (robot description, xacro)
@@ -10,8 +10,5 @@
       <origin rpy="0 0 0" xyz="0.00000000 0.00000000 0.00208424"/>
       <mass value="0.11166745"/>
-      <inertia
-        ixx="0.004391"
-        ixy="0.000000" iyy="0.004391"
-        ixz="0.000000" iyz="0.000000" izz="0.004277"/>
+      <inertia ixx="0.004391" ixy="0.000000" iyy="0.004391" ixz="0.000000" iyz="0.000000" izz="0.004277"/>
     </inertial>
     <visual>

Commit message: wip

File: cube_petit_description/xacro/cube_petit_gazebo.xacro (robot description, xacro)
@@ -240,10 +240,37 @@
     </collision>
   </link>
+  <joint name="camera_optical_joint" type="fixed">
+    <parent link="camera_link"/>
+    <child link="camera_rgb_optical_frame"/>
+    <origin rpy="-1.57 0 -1.57" xyz="0.0 0.0 0.0"/>
+  </joint>
+  <link name="camera_rgb_optical_frame">
+    <inertial>
+      <origin rpy="0 0 0" xyz="0.00000000 0.00000000 0.0000000"/>
+      <mass value="0.11166745"/>
+      <inertia ixx="0.004391" ixy="0.000000" iyy="0.004391" ixz="0.000000" iyz="0.000000" izz="0.004277"/>
+    </inertial>
+    <visual>
+      <origin rpy="0 0 0" xyz="0 0 0"/>
+      <geometry>
+        <cylinder length="0.001" radius="0.001"/>
+      </geometry>
+      <!-- <material name="red">
+        <color rgba="1.0 0.0 0.0 1.0"/>
+      </material> -->
+    </visual>
+    <collision>
+      <origin rpy="0 0 0" xyz="0 0 0"/>
+      <geometry>
+        <cylinder length="0.001" radius="0.001"/>
+      </geometry>
+    </collision>
+  </link>
   <joint name="depth_optical_joint" type="fixed">
-    <parent link="camera_link"/>
-    <child link="camera_optical_link"/>
-    <origin rpy="-1.57 0 -1.57" xyz="0.0 0.0 0.0"/>
-  </joint>
-  <link name="camera_optical_link">
+    <parent link="camera_rgb_optical_frame"/>
+    <child link="camera_depth_optical_frame"/>
+    <origin rpy="0 0 0" xyz="0.0 0.0 0.0"/>
+  </joint>
+  <link name="camera_depth_optical_frame">
     <inertial>
       <origin rpy="0 0 0" xyz="0.00000000 0.00000000 0.0000000"/>
@@ -272,5 +299,5 @@
       <update_rate>4.0</update_rate>
       <topic>camera/depth/image_raw</topic>
-      <frame>camera_optical_link</frame>
+      <frame>camera_depth_optical_frame</frame>
       <camera>
         <camera_info_topic>camera/depth/camera_info</camera_info_topic>
@@ -291,5 +318,5 @@
       <update_rate>4.0</update_rate>
       <topic>camera/rgb/image_raw</topic>
-      <frame>camera_optical_link</frame>
+      <frame>camera_rgb_optical_frame</frame>
       <camera>
         <camera_info_topic>camera/rgb/camera_info</camera_info_topic>
@@ -307,5 +334,5 @@
       <!-- <plugin name="gz::sim::systems::Sensors" filename="gz-sim-sensors-system">
         <output_type>sensor_msgs/CameraInfo</output_type>
-        <frame_name>camera_optical_link</frame_name>
+        <frame_name>rgb_optical_frame</frame_name>
       </plugin> -->
     </sensor>

Commit message: add navigation

File: cube_petit_description/xacro/cube_petit_gazebo.xacro (robot description, xacro)
@@ -1,3 +1,3 @@
-<?xml version="1.0"?>
+<?xml version="1.0" encoding="UTF-8"?>
 <robot xmlns:xacro="http://www.ros.org/wiki/xacro" name="cube_petit_v3">
   <!-- General -->
@@ -7,4 +7,10 @@
   <xacro:include filename="$(find
   cube_petit_description)/xacro/brass_gazebo_battery/brass_gazebo_battery.xacro"/> -->
+  <link name="base_footprint"/>
+  <joint name="base_joint" type="fixed">
+    <parent link="base_footprint"/>
+    <child link="base_link"/>
+    <origin xyz="0.0 0.0 0.0" rpy="0.0 0.0 0.0"/>
+  </joint>
   <link name="base_link"/>
   <joint name="body_joint" type="fixed">
@@ -93,6 +99,6 @@
       <always_on>true</always_on>
       <visualize>false</visualize>
-      <update_rate>10</update_rate>
-      <topic>/pacecat/scan</topic>
+      <update_rate>5</update_rate>
+      <topic>/laser/scan</topic>
       <gz_frame_id>pacecat_link</gz_frame_id>
       <lidar>
@@ -291,5 +297,5 @@
       <update_rate>4.0</update_rate>
       <topic>camera/rgb/image_raw</topic>
-      <gz_frame_id>camera_rbg_optical_frame</gz_frame_id>
+      <gz_frame_id>camera_color_optical_link</gz_frame_id>
       <camera>
         <camera_info_topic>camera/rgb/camera_info</camera_info_topic>

File: cube_petit_description/xacro/sensors/lidar.xacro (robot description, xacro)
@@ -58,5 +58,5 @@
         <ros>
           <namespace>/pacecat</namespace>
-          <remapping>~/out:=/pacecat/scan</remapping>
+          <remapping>~/out:=/laser/scan</remapping>
         </ros>
         <output_type>sensor_msgs/LaserScan</output_type>
