Commit message: update real sense bring up

File: cube_petit_description/xacro/cube_petit.xacro (robot description, xacro)
@@ -60,4 +60,58 @@
   </joint>
   <xacro:include filename="$(find cube_petit_description)/xacro/sensors/lidar.xacro"/>
+  <joint name="depth_joint" type="fixed">
+    <parent link="body_link"/>
+    <child link="camera_link"/>
+    <origin rpy="0 0.0034 0" xyz="0.10137 -0.006 0.097793"/>
+  </joint>
+  <link name="camera_link">
+    <inertial>
+      <origin rpy="0 0 0" xyz="0.00000000 0.00000000 0.0000000"/>
+      <mass value="0.11166745"/>
+      <inertia ixx="0.004391" ixy="0.000000" iyy="0.004391" ixz="0.000000" iyz="0.000000" izz="0.004277"/>
+    </inertial>
+    <visual>
+      <origin rpy="0 0 0" xyz="0 0 0"/>
+      <geometry>
+        <cylinder length="0.001" radius="0.001"/>
+      </geometry>
+      <!-- <material name="red">
+        <color rgba="1.0 0.0 0.0 1.0"/>
+      </material> -->
+    </visual>
+    <collision>
+      <origin rpy="0 0 0" xyz="0 0 0"/>
+      <geometry>
+        <cylinder length="0.001" radius="0.001"/>
+      </geometry>
+    </collision>
+  </link>
+  <joint name="depth_optical_joint" type="fixed">
+    <parent link="camera_link"/>
+    <child link="camera_depth_optical_frame"/>
+    <origin rpy="-1.57 0 -1.57" xyz="0.0 0.0 0.0"/>
+  </joint>
+  <link name="camera_depth_optical_frame">
+    <inertial>
+      <origin rpy="0 0 0" xyz="0.00000000 0.00000000 0.0000000"/>
+      <mass value="0.11166745"/>
+      <inertia ixx="0.004391" ixy="0.000000" iyy="0.004391" ixz="0.000000" iyz="0.000000" izz="0.004277"/>
+    </inertial>
+    <visual>
+      <origin rpy="0 0 0" xyz="0 0 0"/>
+      <geometry>
+        <cylinder length="0.001" radius="0.001"/>
+      </geometry>
+      <!-- <material name="red">
+        <color rgba="1.0 0.0 0.0 1.0"/>
+      </material> -->
+    </visual>
+    <collision>
+      <origin rpy="0 0 0" xyz="0 0 0"/>
+      <geometry>
+        <cylinder length="0.001" radius="0.001"/>
+      </geometry>
+    </collision>
+  </link>
   <!-- rear camera -->
   <!-- <xacro:include filename="$(find cube_petit_description)/xacro/sensors/camera.xacro" /> -->

Commit message: update orange

File: cube_petit_description/xacro/cube_petit.xacro (robot description, xacro)
@@ -7,7 +7,7 @@
   <xacro:include filename="$(find
   cube_petit_description)/xacro/brass_gazebo_battery/brass_gazebo_battery.xacro"/> -->
-  <link name="base_link"/>
+  <link name="cube_petit_orange/base_link"/>
   <joint name="body_joint" type="fixed">
-    <parent link="base_link"/>
+    <parent link="cube_petit_orange/base_link"/>
     <child link="body_link"/>
     <origin rpy="0 0 0" xyz="0 0 0"/>
@@ -15,5 +15,5 @@
   <link name="base_link_reverse"/>
   <joint name="base_link_reverse_joint" type="fixed">
-    <parent link="base_link"/>
+    <parent link="cube_petit_orange/base_link"/>
     <child link="base_link_reverse"/>
     <origin rpy="0 0 3.1415926" xyz="0 0 0"/>
@@ -21,5 +21,5 @@
   <link name="respeaker_base"/>
   <joint name="respeaker_joint" type="fixed">
-    <parent link="base_link"/>
+    <parent link="cube_petit_orange/base_link"/>
     <child link="respeaker_base"/>
     <origin rpy="0 0 0" xyz="0 0 0.28"/>
@@ -55,5 +55,5 @@
   <link name="connector_link"/>
   <joint name="connector_joint" type="fixed">
-    <parent link="base_link"/>
+    <parent link="cube_petit_orange/base_link"/>
     <child link="connector_link"/>
     <origin rpy="0 0 3.14" xyz="-0.11 0 0.025"/>
