Commit message: fix: URDFのroot link名をcube_petit_orange固定からhostname由来の名前空間へ
cube_petit.xacroがcube_petit_orange/base_linkをハードコードしていたため、
pink等の他機体でもrobot_state_publisherが常にorange名義のTFを発行していた。
これがnavigation側のTFツリー(<robot>/base_link起点)と接続せず、地図が
表示されない(slam_toolboxのmessage filterがqueue full)root causeだった。

xacro側にrobot_namespace引数を追加し、cube_petit_bringup.launch.pyの
hostname由来のnsをそこへ渡すよう配線。cube_petit_control.launch.pyは
既に宣言だけされていた同名の未使用引数を実際に配線した。

File: cube_petit_description/xacro/cube_petit.xacro (robot description, xacro)
@@ -7,7 +7,15 @@
   <xacro:include filename="$(find
   cube_petit_description)/xacro/brass_gazebo_battery/brass_gazebo_battery.xacro"/> -->
-  <link name="cube_petit_orange/base_link"/>
+  <!-- robot_namespace: hostnameから自動導出される名前空間(cube_petit_orange/pink/...)。
+       navigation.launch.py等が期待するroot link名(<robot>/base_link)に合わせるため、
+       ここをハードコードせずxacro引数として受け取る(2026-07-27)。
+       robot_namespace: the namespace auto-derived from hostname (cube_petit_orange/pink/...).
+       Kept as an xacro arg (default cube_petit_orange) instead of a hardcoded literal so the
+       root link name (<robot>/base_link) matches what navigation.launch.py etc. expect. -->
+  <xacro:arg name="robot_namespace" default="cube_petit_orange"/>
+  <xacro:property name="robot_ns" value="$(arg robot_namespace)"/>
+  <link name="${robot_ns}/base_link"/>
   <joint name="body_joint" type="fixed">
-    <parent link="cube_petit_orange/base_link"/>
+    <parent link="${robot_ns}/base_link"/>
     <child link="body_link"/>
     <origin rpy="0 0 0" xyz="0 0 0"/>
@@ -15,5 +23,5 @@
   <link name="base_link_reverse"/>
   <joint name="base_link_reverse_joint" type="fixed">
-    <parent link="cube_petit_orange/base_link"/>
+    <parent link="${robot_ns}/base_link"/>
     <child link="base_link_reverse"/>
     <origin rpy="0 0 3.1415926" xyz="0 0 0"/>
@@ -21,5 +29,5 @@
   <link name="respeaker_base"/>
   <joint name="respeaker_joint" type="fixed">
-    <parent link="cube_petit_orange/base_link"/>
+    <parent link="${robot_ns}/base_link"/>
     <child link="respeaker_base"/>
     <origin rpy="0 0 0" xyz="0 0 0.28"/>
@@ -55,5 +63,5 @@
   <link name="connector_link"/>
   <joint name="connector_joint" type="fixed">
-    <parent link="cube_petit_orange/base_link"/>
+    <parent link="${robot_ns}/base_link"/>
     <child link="connector_link"/>
     <origin rpy="0 0 3.14" xyz="-0.11 0 0.025"/>
